File: hardware/kicad/nightwave-reference/06_connectors_test.kicad_sch (KiCad schematic)
At the start: 14 parts, among them J8 UART0_SERVICE, SW6 MAIN_POWER

Commit message: hardware: close reference PCB routing and verify CAD exports
Parts:
- added TP13: BT_SERVICE_P34, TestPoint:TestPoint_Pad_D1.0mm, symbol Nightwave:TP13
- added TP14: BT_LED, TestPoint:TestPoint_Pad_D1.0mm, symbol Nightwave:TP14
- added TP15: BT_STATE, TestPoint:TestPoint_Pad_D1.0mm, symbol Nightwave:TP15
- added TP16: HP_DETECT, TestPoint:TestPoint_Pad_D1.0mm, symbol Nightwave:TP16
- J8: symbol Connector_Generic:Conn_01x06 -> Nightwave:J8
- SW6: symbol Switch:SW_SPDT -> Nightwave:SW6
- TP1: symbol Connector:TestPoint -> Nightwave:TP1
- TP10: symbol Connector:TestPoint -> Nightwave:TP10
- TP11: symbol Connector:TestPoint -> Nightwave:TP11
- TP12: symbol Connector:TestPoint -> Nightwave:TP12
- TP2: symbol Connector:TestPoint -> Nightwave:TP2
- TP3: symbol Connector:TestPoint -> Nightwave:TP3
- TP4: symbol Connector:TestPoint -> Nightwave:TP4
- TP5: symbol Connector:TestPoint -> Nightwave:TP5
- TP6: symbol Connector:TestPoint -> Nightwave:TP6
- TP7: symbol Connector:TestPoint -> Nightwave:TP7
- TP8: symbol Connector:TestPoint -> Nightwave:TP8
- TP9: symbol Connector:TestPoint -> Nightwave:TP9
Connections:
- net +3V3: now also J8.1 (Pin_1); no longer J8.5 (Pin_5)
- net BOOT_N: now also J8.6 (Pin_6)
- net ESP_EN: now also J8.5 (Pin_5); no longer J8.1 (Pin_1)
- net GND: now also J8.2 (Pin_2), SW6.1 (A); no longer J8.4 (Pin_4), SW6.3 (C)
- net SYS: now also SW6.3 (C); no longer SW6.1 (A)
- net UART0_RX: now also J8.4 (Pin_4); no longer J8.2 (Pin_2)
- new net BT_LED: TP14.1
- new net BT_SERVICE_P34: TP13.1
- new net BT_STATE: TP15.1
- new net HP_DETECT: TP16.1
Other:
- moved on the sheet: J8
