File: hardware/kicad/nightwave-reference/01_power_charging.kicad_sch (KiCad schematic)
At the start: 21 parts, among them J1 USB4105-GF-A, J2 BATTERY_1S_10050mAh, J3 EXTERNAL_10K_NTC, U2 TUSB320LAIRWBR, U3 BQ25628ERYKR, U4 TPS22965DSGR, U5 TPS63802DLAR, U6 TPS63802DLAR, U7 MAX17048G+T10

Commit message: hardware: close reference PCB routing and verify CAD exports
Parts:
- removed U2: TUSB320LAIRWBR, Package_DFN_QFN:Texas_X2QFN-12_1.6x1.6mm_P0.4mm, symbol Connector_Generic:Conn_01x12
- added C10: 10u/25V, Capacitor_SMD:C_0805_2012Metric, symbol Nightwave:C10
- added C11: 10u/10V, Capacitor_SMD:C_0805_2012Metric, symbol Nightwave:C11
- added C12: 22u/10V, Capacitor_SMD:C_0805_2012Metric, symbol Nightwave:C12
- added C13: 10u/10V, Capacitor_SMD:C_0805_2012Metric, symbol Nightwave:C13
- added C14: 22u/10V, Capacitor_SMD:C_0805_2012Metric, symbol Nightwave:C14
- added C15: 100n/10V, Capacitor_SMD:C_0805_2012Metric, symbol Nightwave:C15
- added C9: 47n/10V, Capacitor_SMD:C_0805_2012Metric, symbol Nightwave:C9
- added L1: 0.47uH XFL4015-471MEC, Nightwave:Coilcraft_XFL4015, symbol Nightwave:L1
- added L2: 0.47uH XFL4015-471MEC, Nightwave:Coilcraft_XFL4015, symbol Nightwave:L2
- added L3: 0.7uH XFL4015-701MEC, Nightwave:Coilcraft_XFL4015, symbol Nightwave:L3
- added R16: 511k, Resistor_SMD:R_0603_1608Metric, symbol Nightwave:R16
- added R17: 91k, Resistor_SMD:R_0603_1608Metric, symbol Nightwave:R17
- added R18: 562k, Resistor_SMD:R_0603_1608Metric, symbol Nightwave:R18
- added R19: 91k, Resistor_SMD:R_0603_1608Metric, symbol Nightwave:R19
- added R20: 5.49k, Resistor_SMD:R_0603_1608Metric, symbol Nightwave:R20
- added R21: 5.23k, Resistor_SMD:R_0603_1608Metric, symbol Nightwave:R21
- added R22: 30.1k, Resistor_SMD:R_0603_1608Metric, symbol Nightwave:R22
- added R23: 0, Resistor_SMD:R_0603_1608Metric, symbol Nightwave:R23
- C1: symbol Device:C -> Nightwave:C1
- C2: symbol Device:C -> Nightwave:C2
- C3: symbol Device:C -> Nightwave:C3
- C4: symbol Device:C -> Nightwave:C4
- C5: symbol Device:C -> Nightwave:C5
- C6: symbol Device:C -> Nightwave:C6
- C7: symbol Device:C -> Nightwave:C7
- C8: value 1u -> 4.7u; symbol Device:C -> Nightwave:C8
- J1: symbol Connector:USB_C_Receptacle_USB2.0_16P -> Nightwave:J1
- J2: value BATTERY_1S_10050mAh -> BATTERY_CONNECTOR; symbol Connector_Generic:Conn_01x02 -> Nightwave:J2
- J3: symbol Connector_Generic:Conn_01x02 -> Nightwave:J3
- R1: symbol Device:R -> Nightwave:R1
- R2: symbol Device:R -> Nightwave:R2
- R3: symbol Device:R -> Nightwave:R3
- R4: symbol Device:R -> Nightwave:R4
- U3: footprint Package_DFN_QFN:WQFN-24-1EP_4x4mm_P0.5mm_EP2.6x2.6mm_ThermalVias -> Nightwave:TI_RYK0018A; symbol Connector_Generic:Conn_01x25 -> Nightwave:U3
- U4: symbol Connector_Generic:Conn_01x09 -> Nightwave:U4
- U5: footprint Package_DFN_QFN:Texas_DSQ0010A_WSON-10-1EP_2x2mm_P0.4mm_EP0.9x1.5mm_ThermalVias -> Nightwave:TI_DLA0010A; symbol Connector_Generic:Conn_01x11 -> Nightwave:U5
- U6: footprint Package_DFN_QFN:Texas_DSQ0010A_WSON-10-1EP_2x2mm_P0.4mm_EP0.9x1.5mm_ThermalVias -> Nightwave:TI_DLA0010A; symbol Connector_Generic:Conn_01x11 -> Nightwave:U6
- U7: symbol Connector_Generic:Conn_01x09 -> Nightwave:U7
Connections:
- net +3V3: now also R3.2 (+3V3), R4.2 (+3V3), C12.1 (+3V3), R16.1 (+3V3); no longer C1.1, C1.2, C2.1, C2.2, C3.1, C3.2, C4.1, C4.2, C5.2, C6.1, C7.1, C8.1, C8.2, J1.B8 (SBU2), J2.1 (Pin_1), J3.1 (Pin_1), R1.1, R1.2, R2.1, R2.2, R3.1, R4.1, U3.1 (Pin_1), U3.10 (Pin_10), U3.16 (Pin_16), U3.17 (Pin_17), U3.18 (Pin_18), U3.19 (Pin_19), U3.2 (Pin_2), U3.20 (Pin_20), U3.21 (Pin_21), U3.22 (Pin_22), U3.23 (Pin_23), U3.24 (Pin_24), U3.25 (Pin_25), U3.3 (Pin_3), U3.4 (Pin_4), U3.5 (Pin_5), U3.6 (Pin_6), U3.7 (Pin_7), U3.8 (Pin_8), U3.9 (Pin_9), U4.1 (Pin_1), U4.2 (Pin_2), U4.3 (Pin_3), U4.4 (Pin_4), U4.5 (Pin_5), U4.6 (Pin_6), U4.8 (Pin_8), U4.9 (Pin_9), U5.1 (Pin_1), U5.10 (Pin_10), U5.11 (Pin_11), U5.2 (Pin_2), U5.3 (Pin_3), U5.5 (Pin_5), U5.8 (Pin_8), U5.9 (Pin_9), U6.1 (Pin_1), U6.10 (Pin_10), U6.11 (Pin_11), U6.2 (Pin_2), U6.3 (Pin_3), U6.8 (Pin_8), U6.9 (Pin_9), U7.1 (Pin_1), U7.2 (Pin_2), U7.3 (Pin_3), U7.4 (Pin_4), U7.8 (Pin_8), U7.9 (Pin_9)
- net +3V3_A: now also C7.1 (+3V3_A); no longer C7.2
- net +3V6_BT: now also C6.1 (+3V6_BT), C14.1 (+3V6_BT), R18.1 (+3V6_BT); no longer C6.2, U6.5 (Pin_5)
- net CHASSIS: now also J1.SH (SHIELD), R23.1 (CHASSIS)
- net CHG_INT_N: now also U3.11 (INT); no longer U3.12 (Pin_12)
- net CHG_STAT: now also U3.10 (STAT); no longer U3.11 (Pin_11)
- net FB_3V3: now also U5.4 (FB), R16.2 (FB_3V3), R17.1 (FB_3V3); no longer U5.7 (Pin_7)
- net FB_BT: now also U6.4 (FB), R18.2 (FB_BT), R19.1 (FB_BT); no longer U6.7 (Pin_7)
- net I2C_SCL: now also R4.1 (I2C_SCL); no longer R4.2
- net I2C_SDA: now also R3.1 (I2C_SDA), U3.12 (SDA), U7.8 (SDA); no longer R3.2, U3.14 (Pin_14), U7.6 (Pin_6)
- net ILIM: now also U3.4 (ILIM), R20.1 (ILIM); no longer U3.15 (Pin_15)
- net PWR_GOOD_3V3: now also U5.5 (PG); no longer U5.4 (Pin_4)
- net PWR_GOOD_BT: now also U6.5 (PG); no longer U6.4 (Pin_4)
- net PWR_SWITCH_ON: now also U4.3 (ON); no longer U4.7 (Pin_7)
- net USB_DM: now also J1.A7 (D-); no longer J1.A6 (D+)
- net USB_DP: now also J1.A6 (D+), J1.B6 (D+); no longer J1.A7 (D-)
- net GND: now reaches J2.2 (Pin_2)
- net GND: now also C1.2 (GND), C2.2 (GND), C3.2 (GND), C4.2 (GND), C5.2 (GND), C6.2 (GND), C7.2 (GND), C8.2 (GND), J1.A1 (GND), J1.A12 (GND), J1.B1 (GND), J1.B12 (GND), J3.2 (Pin_2), R1.2 (GND), R2.2 (GND), U3.14 (CE), U3.15 (GND), U4.5 (GND), U4.9 (EP), U5.2 (MODE), U5.3 (AGND), U5.8 (GND), U6.2 (MODE), U6.3 (AGND), U6.8 (GND), U7.1 (CTG), U7.4 (GND), U7.6 (QSTRT), U7.9 (EP), C10.2 (GND), C11.2 (GND), C12.2 (GND), C13.2 (GND), C14.2 (GND), C15.2 (GND), R17.2 (GND), R19.2 (GND), R20.2 (GND), R22.2 (GND), R23.2 (GND)
- net VBUS5: now reaches J1.A4 (VBUS), J1.A9 (VBUS), J1.B4 (VBUS), J1.B9 (VBUS)
- net VBUS5: now also C1.1 (VBUS5), U3.18 (VBUS)
- net USB_CC1: now reaches J1.A5 (CC1)
- net USB_CC1: now also R1.1 (USB_CC1)
- net USB_CC2: now reaches J1.B5 (CC2)
- net USB_CC2: now also R2.1 (USB_CC2)
- new net BAT: C15.1 (BAT), C2.1 (BAT), J2.1 (Pin_1), U3.8 (BAT), U7.2 (CELL), U7.3 (VDD)
- new net BTST: C9.1 (BTST), U3.1 (BTST)
- new net PGOOD_CHG: U3.3 (PG)
- new net PMID: C10.1 (PMID), U3.17 (PMID)
- new net REGN: C8.1 (REGN), U3.2 (REGN)
- new net SW1_3V3: L1.1, U5.9 (L1)
- new net SW1_BT: L2.1, U6.9 (L1)
- new net SW2_3V3: L1.2, U5.7 (L2)
- new net SW2_BT: L2.2, U6.7 (L2)
- new net SW_CHG: C9.2 (SW_CHG), L3.1, U3.16 (SW)
- new net SYS: C3.1 (SYS), L3.2, U3.9 (SYS), U4.1 (VIN), U4.2 (VIN), U4.4 (VBIAS)
- new net TS: J3.1 (Pin_1), R21.2 (TS), R22.1 (TS), U3.6 (TS)
- new net TS_BIAS: R21.1 (TS_BIAS), U3.5 (TS_BIAS)
- new net VSYS_SW: C11.1 (VSYS_SW), C13.1 (VSYS_SW), C4.1 (VSYS_SW), U4.7 (VOUT), U4.8 (VOUT), U5.1 (EN), U5.10 (VIN), U6.1 (EN), U6.10 (VIN)
- no-connect marks 2 -> 4
Other:
- moved on the sheet: J2, J3, U4, U7
