File: hardware/kicad/nightwave-reference/02_mcu_storage.kicad_sch (KiCad schematic)
At the start: 4 parts, among them J4 Molex 104031-0811, U1 ESP32-S3-WROOM-1-N16R8

Commit message: hardware: close reference PCB routing and verify CAD exports
Parts:
- added C16: 100n/10V, Capacitor_SMD:C_0805_2012Metric, symbol Nightwave:C16
- added C17: 10u/10V, Capacitor_SMD:C_0805_2012Metric, symbol Nightwave:C17
- added C18: 1u/10V, Capacitor_SMD:C_0805_2012Metric, symbol Nightwave:C18
- added C19: 100n/10V, Capacitor_SMD:C_0805_2012Metric, symbol Nightwave:C19
- added C20: 10u/10V, Capacitor_SMD:C_0805_2012Metric, symbol Nightwave:C20
- added R24: 10k, Resistor_SMD:R_0603_1608Metric, symbol Nightwave:R24
- added R25: 10k, Resistor_SMD:R_0603_1608Metric, symbol Nightwave:R25
- added R48: 10k, Resistor_SMD:R_0603_1608Metric, symbol Nightwave:R48
- added R49: 10k, Resistor_SMD:R_0603_1608Metric, symbol Nightwave:R49
- added R50: 10k, Resistor_SMD:R_0603_1608Metric, symbol Nightwave:R50
- J4: symbol Connector:Micro_SD_Card -> Nightwave:J4
- R5: symbol Device:R -> Nightwave:R5
- R6: symbol Device:R -> Nightwave:R6
- U1: symbol Connector_Generic:Conn_01x41 -> Nightwave:U1
Connections:
- net SD_D2_NC is gone; now on net SD_D0: J4.7 (DAT0)
- net +3V3: now also C16.1 (+3V3), C17.1 (+3V3), C19.1 (+3V3), C20.1 (+3V3), R24.2 (+3V3), R25.2 (+3V3), R48.2 (+3V3), R49.2 (+3V3), R50.2 (+3V3); no longer J4.2 (DAT3/CD), J4.6 (VSS), U1.1 (Pin_1), U1.3 (Pin_3), U1.30 (Pin_30), U1.31 (Pin_31), U1.32 (Pin_32), U1.33 (Pin_33), U1.34 (Pin_34), U1.35 (Pin_35), U1.36 (Pin_36), U1.37 (Pin_37), U1.38 (Pin_38), U1.39 (Pin_39), U1.4 (Pin_4), U1.40 (Pin_40), U1.41 (Pin_41)
- net BOOT_N: now also U1.27 (GPIO0), R25.1 (BOOT_N); no longer U1.14 (Pin_14), U1.15 (Pin_15)
- net BT_MCLK_OPTION: now also U1.23 (GPIO21); no longer U1.19 (Pin_19)
- net BT_WAKE: now also U1.18 (GPIO10); no longer U1.24 (Pin_24), U1.25 (Pin_25), U1.26 (Pin_26)
- net HP_EN: now also U1.32 (GPIO39); no longer U1.10 (Pin_10), U1.11 (Pin_11), U1.6 (Pin_6), U1.7 (Pin_7), U1.8 (Pin_8), U1.9 (Pin_9)
- net SD_CLK: now also J4.5 (CLK), U1.20 (GPIO12); no longer J4.3 (CMD), U1.22 (Pin_22)
- net SD_CMD: now also J4.3 (CMD), U1.19 (GPIO11), R48.1 (SD_CMD); no longer J4.5 (CLK), U1.23 (Pin_23)
- net SD_D0: now also R49.1 (SD_D0); no longer J4.1 (DAT2)
- net TCA_INT_N: now also U1.22 (GPIO14); no longer U1.20 (Pin_20)
- net TFT_MOSI: now also U1.24 (GPIO47); no longer U1.16 (Pin_16), U1.17 (Pin_17), U1.18 (Pin_18)
- net USB_DM: now also R6.1 (USB_DM); no longer R6.2
- net USB_DM_MCU: now also R6.2 (USB_DM_MCU), U1.13 (GPIO19_USB_D-); no longer R6.1
- net USB_DP: now also R5.1 (USB_DP); no longer R5.2
- net USB_DP_MCU: now also R5.2 (USB_DP_MCU), U1.14 (GPIO20_USB_D+); no longer R5.1
- net GND: now reaches J4.SH (SHIELD)
- net GND: now also J4.10 (GND), J4.6 (VSS), U1.1 (GND), U1.40 (GND), U1.41 (EP_GND), C16.2 (GND), C17.2 (GND), C18.2 (GND), C19.2 (GND), C20.2 (GND)
- net I2C_SDA: now reaches U1.12 (GPIO8)
- net I2S_BCLK: now reaches U1.5 (GPIO5)
- new net BT_MFB: U1.4 (GPIO4)
- new net BT_RST_N: U1.8 (GPIO15)
- new net BT_UART_RX: U1.38 (GPIO2)
- new net BT_UART_TX: U1.39 (GPIO1)
- new net DAC_XSMT: U1.11 (GPIO18)
- new net ESP_EN: C18.1 (ESP_EN), R24.1 (ESP_EN), U1.3 (EN)
- new net HP_DETECT: U1.9 (GPIO16)
- new net I2C_SCL: U1.17 (GPIO9)
- new net I2S_DOUT: U1.7 (GPIO7)
- new net I2S_LRCLK: U1.6 (GPIO6)
- new net SD_DAT3: J4.2 (DAT3/CD), R50.1 (SD_DAT3)
- new net SD_DETECT_N: J4.9 (SD_DETECT_N)
- new net SPK_EN: U1.10 (GPIO17)
- new net TFT_BL_PWM: U1.31 (GPIO38)
- new net TFT_CS: U1.35 (GPIO42)
- new net TFT_DC: U1.34 (GPIO41)
- new net TFT_RST: U1.33 (GPIO40)
- new net TFT_SCLK: U1.25 (GPIO48)
- new net UART0_RX: U1.36 (RXD0)
- new net UART0_TX: U1.37 (TXD0)
- no-connect marks 10 -> 8
Other:
- moved on the sheet: U1
