File: hardware/kicad/nightwave-reference/03_local_audio.kicad_sch (KiCad schematic)
At the start: 11 parts, among them J5 SJ-3523-SMT-TR, J6 CMS-28528N-L152, U10 MAX98357AETE+T, U8 PCM5102APWR, U9 TPA6132A2RTER

Commit message: hardware: close reference PCB routing and verify CAD exports
Parts:
- added C21: 2.2u/10V, Capacitor_SMD:C_0805_2012Metric, symbol Nightwave:C21
- added C22: 2.2u/10V, Capacitor_SMD:C_0805_2012Metric, symbol Nightwave:C22
- added C23: 100n/10V, Capacitor_SMD:C_0805_2012Metric, symbol Nightwave:C23
- added C24: 100n/10V, Capacitor_SMD:C_0805_2012Metric, symbol Nightwave:C24
- added C25: 100n/10V, Capacitor_SMD:C_0805_2012Metric, symbol Nightwave:C25
- added C26: 1u/10V, Capacitor_SMD:C_0805_2012Metric, symbol Nightwave:C26
- added C27: 1u/10V, Capacitor_SMD:C_0805_2012Metric, symbol Nightwave:C27
- added C28: 2.2u/10V, Capacitor_SMD:C_0805_2012Metric, symbol Nightwave:C28
- added C29: 1u/10V, Capacitor_SMD:C_0805_2012Metric, symbol Nightwave:C29
- added C30: 1u/10V, Capacitor_SMD:C_0805_2012Metric, symbol Nightwave:C30
- added C31: 100n/10V, Capacitor_SMD:C_0805_2012Metric, symbol Nightwave:C31
- added C32: 100n/10V, Capacitor_SMD:C_0805_2012Metric, symbol Nightwave:C32
- added C33: 10u/10V, Capacitor_SMD:C_0805_2012Metric, symbol Nightwave:C33
- added R27: 10k, Resistor_SMD:R_0603_1608Metric, symbol Nightwave:R27
- added R28: 10k, Resistor_SMD:R_0603_1608Metric, symbol Nightwave:R28
- added R29: 10k, Resistor_SMD:R_0603_1608Metric, symbol Nightwave:R29
- added R30: 0, Resistor_SMD:R_0603_1608Metric, symbol Nightwave:R30
- added R51: 47k, Resistor_SMD:R_0603_1608Metric, symbol Nightwave:R51
- J5: value SJ-3523-SMT-TR -> SJ3-350153AG-TR; footprint Connector_Audio:Jack_3.5mm_CUI_SJ-3523-SMT_Horizontal -> Nightwave:SameSky_SJ3-350153AG; symbol Connector_Audio:AudioJack3_Ground_Switch -> Nightwave:J5
- J6: value CMS-28528N-L152 -> BTL_SPEAKER_CONNECTOR; symbol Connector_Generic:Conn_01x02 -> Nightwave:J6
- R10: symbol Device:R -> Nightwave:R10
- R11: symbol Device:R -> Nightwave:R11
- R12: symbol Device:R -> Nightwave:R12
- R7: symbol Device:R -> Nightwave:R7
- R8: symbol Device:R -> Nightwave:R8
- R9: symbol Device:R -> Nightwave:R9
- U10: footprint Package_CSP:WLCSP-9_1.21x1.22mm_Layout3x3_P0.4mm -> Package_DFN_QFN:TQFN-16-1EP_3x3mm_P0.5mm_EP1.23x1.23mm; symbol Audio:MAX98357A -> Nightwave:U10
- U8: symbol Connector_Generic:Conn_01x20 -> Nightwave:U8
- U9: symbol Connector_Generic:Conn_01x17 -> Nightwave:U9
Connections:
- net +3V3: now also C25.1 (+3V3), R30.1 (+3V3); no longer J5.RN, J5.S, J5.T, R7.1, R8.1, R9.1, U10.16 (BCLK), U8.1 (Pin_1), U8.10 (Pin_10), U8.11 (Pin_11), U8.12 (Pin_12), U8.17 (Pin_17), U8.18 (Pin_18), U8.19 (Pin_19), U8.2 (Pin_2), U8.3 (Pin_3), U8.4 (Pin_4), U8.5 (Pin_5), U8.6 (Pin_6), U8.7 (Pin_7), U8.8 (Pin_8), U8.9 (Pin_9), U9.1 (Pin_1), U9.10 (Pin_10), U9.2 (Pin_2), U9.3 (Pin_3), U9.4 (Pin_4), U9.5 (Pin_5), U9.8 (Pin_8)
- net DAC_L: now also U8.6 (OUTL), C29.1 (DAC_L); no longer J5.R, U8.13 (Pin_13), U8.14 (Pin_14), U8.15 (Pin_15), U9.13 (Pin_13), U9.14 (Pin_14), U9.15 (Pin_15), U9.16 (Pin_16), U9.17 (Pin_17)
- net HP_DETECT: now also J5.6 (Pin_6)
- net I2S_BCLK: now also R10.1 (I2S_BCLK), R7.1 (I2S_BCLK); no longer R10.2, R7.2
- net I2S_BCLK_SPK: now also R10.2 (I2S_BCLK_SPK), U10.16 (BCLK); no longer R10.1, U10.2 (GAIN_SLOT)
- net I2S_DOUT: now also R12.1 (I2S_DOUT), R9.1 (I2S_DOUT); no longer R12.2, R9.2
- net I2S_DOUT_SPK: now also R12.2 (I2S_DOUT_SPK), U10.1 (DIN); no longer R12.1
- net I2S_LRCLK: now also R11.1 (I2S_LRCLK), R8.1 (I2S_LRCLK); no longer R11.2, R8.2
- net I2S_LRCLK_SPK: now also R11.2 (I2S_LRCLK_SPK), U10.14 (LRCLK); no longer R11.1, U10.4 (~{SD_MODE})
- net SPK_EN: now also R51.1 (SPK_EN); no longer U10.14 (LRCLK)
- net SPK_N: now also J6.2 (Pin_2), U10.10 (OUTN)
- net SPK_P: now also U10.9 (OUTP)
- net VSYS_SW: now also U10.7 (VDD), U10.8 (VDD), C32.1 (VSYS_SW), C33.1 (VSYS_SW)
- net GND: now reaches U8.16 (FMT)
- net GND: now also J5.1 (Pin_1), J5.4 (Pin_4), J5.5 (Pin_5), J5.MS (GND), U10.11 (GND), U10.15 (GND), U10.17 (PAD), U10.2 (GAIN_SLOT), U10.3 (GND), U8.10 (DEMP), U8.11 (FLT), U8.12 (SCK), U8.19 (DGND), U8.3 (CPGND), U8.9 (AGND), U9.10 (PGND), U9.15 (SGND), U9.17 (EP), U9.2 (INL+), U9.3 (INR+), U9.6 (G0), U9.7 (G1), C22.2 (GND), C23.2 (GND), C24.2 (GND), C25.2 (GND), C27.2 (GND), C28.2 (GND), C31.2 (GND), C32.2 (GND), C33.2 (GND), R27.2 (GND), R28.2 (GND), R29.2 (GND)
- net HP_CP_P: now reaches U9.11 (CPP)
- net HP_CP_P: now also C26.1 (HP_CP_P)
- net HP_VDD: now reaches U9.12 (HPVDD)
- net HP_VDD: now also C28.1 (HP_VDD)
- net HP_CP_N: now reaches U9.9 (CPN)
- net HP_CP_N: now also C26.2 (HP_CP_N)
- removed net HP_DETECT_BIAS: J5.SN
- new net +3V3_A: C24.1 (+3V3_A), C31.1 (+3V3_A), R30.2 (+3V3_A), U8.1 (CPVDD), U8.8 (AVDD), U9.14 (VDD)
- new net DAC_R: C30.1 (DAC_R), U8.7 (OUTR)
- new net DAC_XSMT: R29.1 (DAC_XSMT), U8.17 (XSMT)
- new net HP_EN: R28.1 (HP_EN), U9.13 (EN)
- new net HP_IN_L: C29.2 (HP_IN_L), U9.1 (INL-)
- new net HP_IN_R: C30.2 (HP_IN_R), U9.4 (INR-)
- new net HP_L: J5.2 (Pin_2), U9.16 (OUTL)
- new net HP_R: J5.3 (Pin_3), U9.5 (OUTR)
- new net HP_VSS: C27.1 (HP_VSS), U9.8 (HPVSS)
- new net I2S_BCLK_DAC: R7.2 (I2S_BCLK_DAC), U8.13 (BCK)
- new net I2S_DOUT_DAC: R9.2 (I2S_DOUT_DAC), U8.14 (DIN)
- new net I2S_LRCLK_DAC: R8.2 (I2S_LRCLK_DAC), U8.15 (LRCK)
- new net PCM_CP_M: C21.2 (PCM_CP_M), U8.4 (CAPM)
- new net PCM_CP_P: C21.1 (PCM_CP_P), U8.2 (CAPP)
- new net PCM_LDOO: C23.1 (PCM_LDOO), U8.18 (LDOO)
- new net PCM_VNEG: C22.1 (PCM_VNEG), U8.5 (VNEG)
- new net SPK_SD_MODE: R27.1 (SPK_SD_MODE), R51.2 (SPK_SD_MODE), U10.4 (~{SD_MODE})
- no-connect marks 14 -> 4
Other:
- moved on the sheet: J6, U8, U9
