File: hardware/kicad/nightwave-reference/04_display_controls.kicad_sch (KiCad schematic)
At the start: 7 parts, among them J7 Waveshare 24382 TFT, SW1 PREV, SW2 PLAY_PAUSE, SW3 NEXT, SW4 VOL_DOWN, SW5 VOL_UP, U11 TCA9535PWR

Commit message: hardware: close reference PCB routing and verify CAD exports
Parts:
- added C34: 100n/10V, Capacitor_SMD:C_0805_2012Metric, symbol Nightwave:C34
- added C35: 10u/10V, Capacitor_SMD:C_0805_2012Metric, symbol Nightwave:C35
- added R26: 10k, Resistor_SMD:R_0603_1608Metric, symbol Nightwave:R26
- added R31: 10k, Resistor_SMD:R_0603_1608Metric, symbol Nightwave:R31
- added R32: 10k, Resistor_SMD:R_0603_1608Metric, symbol Nightwave:R32
- added R33: 10k, Resistor_SMD:R_0603_1608Metric, symbol Nightwave:R33
- added R34: 10k, Resistor_SMD:R_0603_1608Metric, symbol Nightwave:R34
- added R35: 10k, Resistor_SMD:R_0603_1608Metric, symbol Nightwave:R35
- added R36: 10k, Resistor_SMD:R_0603_1608Metric, symbol Nightwave:R36
- added R37: 10k, Resistor_SMD:R_0603_1608Metric, symbol Nightwave:R37
- added R38: 10k, Resistor_SMD:R_0603_1608Metric, symbol Nightwave:R38
- added R39: 10k, Resistor_SMD:R_0603_1608Metric, symbol Nightwave:R39
- added R40: 10k, Resistor_SMD:R_0603_1608Metric, symbol Nightwave:R40
- added R41: 10k, Resistor_SMD:R_0603_1608Metric, symbol Nightwave:R41
- added R42: 10k, Resistor_SMD:R_0603_1608Metric, symbol Nightwave:R42
- added R43: 10k, Resistor_SMD:R_0603_1608Metric, symbol Nightwave:R43
- added R44: 10k, Resistor_SMD:R_0603_1608Metric, symbol Nightwave:R44
- added R45: 10k, Resistor_SMD:R_0603_1608Metric, symbol Nightwave:R45
- added R46: 10k, Resistor_SMD:R_0603_1608Metric, symbol Nightwave:R46
- added R47: 10k, Resistor_SMD:R_0603_1608Metric, symbol Nightwave:R47
- J7: value Waveshare 24382 TFT -> TFT_24382_HARNESS; symbol Connector_Generic:Conn_01x08 -> Nightwave:J7
- SW1: symbol Switch:SW_Push -> Nightwave:SW1
- SW2: symbol Switch:SW_Push -> Nightwave:SW2
- SW3: symbol Switch:SW_Push -> Nightwave:SW3
- SW4: symbol Switch:SW_Push -> Nightwave:SW4
- SW5: symbol Switch:SW_Push -> Nightwave:SW5
- U11: symbol Connector_Generic:Conn_01x24 -> Nightwave:U11
Connections:
- net USB_INT_N is gone; now on net CHG_STAT: U11.10 (P0_6)
- net +3V3: now also J7.1 (Pin_1), C34.1 (+3V3), C35.1 (+3V3), R26.2 (+3V3), R31.2 (+3V3), R32.2 (+3V3), R33.2 (+3V3), R34.2 (+3V3), R35.2 (+3V3), R36.2 (+3V3), R37.2 (+3V3), R38.2 (+3V3), R39.2 (+3V3), R40.2 (+3V3), R41.2 (+3V3), R42.2 (+3V3), R43.2 (+3V3), R44.2 (+3V3), R45.2 (+3V3), R46.2 (+3V3), R47.2 (+3V3); no longer J7.6 (Pin_6), J7.7 (Pin_7), J7.8 (Pin_8), SW1.1, SW1.2, SW2.1, SW2.2, SW3.1, SW3.2, SW4.1, SW4.2, SW5.1, SW5.2, U11.1 (Pin_1), U11.12 (Pin_12), U11.15 (Pin_15), U11.16 (Pin_16), U11.17 (Pin_17), U11.18 (Pin_18), U11.19 (Pin_19), U11.2 (Pin_2), U11.20 (Pin_20), U11.21 (Pin_21), U11.22 (Pin_22), U11.23 (Pin_23), U11.3 (Pin_3), U11.4 (Pin_4), U11.5 (Pin_5), U11.6 (Pin_6), U11.7 (Pin_7), U11.8 (Pin_8), U11.9 (Pin_9)
- net CHG_INT_N: now also U11.13 (P1_0), R39.1 (CHG_INT_N); no longer U11.11 (Pin_11)
- net CHG_STAT: now also R37.1 (CHG_STAT); no longer U11.14 (Pin_14)
- net FUEL_ALERT_N: now also U11.11 (P0_7), R38.1 (FUEL_ALERT_N); no longer U11.13 (Pin_13)
- net TFT_BL_PWM: now also J7.8 (Pin_8); no longer J7.1 (Pin_1)
- net TFT_CS: now also J7.5 (Pin_5); no longer J7.3 (Pin_3)
- net TFT_DC: now also J7.6 (Pin_6); no longer J7.2 (Pin_2)
- net TFT_MOSI: now also J7.3 (Pin_3); no longer J7.5 (Pin_5)
- new net BTN_NEXT_N: R33.1 (BTN_NEXT_N), SW3.1, U11.6 (P0_2)
- new net BTN_PLAY_N: R32.1 (BTN_PLAY_N), SW2.1, U11.5 (P0_1)
- new net BTN_PREV_N: R31.1 (BTN_PREV_N), SW1.1, U11.4 (P0_0)
- new net BTN_VOL_DOWN_N: R34.1 (BTN_VOL_DOWN_N), SW4.1, U11.7 (P0_3)
- new net BTN_VOL_UP_N: R35.1 (BTN_VOL_UP_N), SW5.1, U11.8 (P0_4)
- new net EXP_IN14: R44.1 (EXP_IN14), U11.17 (P1_4)
- new net EXP_IN15: R45.1 (EXP_IN15), U11.18 (P1_5)
- new net EXP_IN16: R46.1 (EXP_IN16), U11.19 (P1_6)
- new net EXP_IN17: R47.1 (EXP_IN17), U11.20 (P1_7)
- new net GND: C34.2 (GND), C35.2 (GND), J7.2 (Pin_2), J7.MP (GND), SW1.2, SW2.2, SW3.2, SW4.2, SW5.2, U11.12 (GND), U11.2 (A1), U11.21 (A0), U11.3 (A2)
- new net HP_DETECT: R26.1 (HP_DETECT)
- new net I2C_SCL: U11.22 (SCL)
- new net I2C_SDA: U11.23 (SDA)
- new net PGOOD_CHG: R40.1 (PGOOD_CHG), U11.14 (P1_1)
- new net PWR_GOOD_3V3: R41.1 (PWR_GOOD_3V3), U11.15 (P1_2)
- new net PWR_GOOD_BT: R42.1 (PWR_GOOD_BT), U11.16 (P1_3)
- new net SD_DETECT_N: R36.1 (SD_DETECT_N), U11.9 (P0_5)
- new net TCA_INT_N: R43.1 (TCA_INT_N), U11.1 (INT)
- new net TFT_RST: J7.7 (Pin_7)
Other:
- moved on the sheet: SW1, SW2, SW3, SW4, SW5, U11
