File: hardware/kicad/nightwave-reference/05_bluetooth.kicad_sch (KiCad schematic)
At the start: 4 parts, among them U12 BM83SM1-00TA

Commit message: hardware: close reference PCB routing and verify CAD exports
Parts:
- added C36: 10u/10V, Capacitor_SMD:C_0805_2012Metric, symbol Nightwave:C36
- added C37: 100n/10V, Capacitor_SMD:C_0805_2012Metric, symbol Nightwave:C37
- R13: symbol Device:R -> Nightwave:R13
- R14: symbol Device:R -> Nightwave:R14
- R15: symbol Device:R -> Nightwave:R15
- U12: footprint RF_Module:Microchip_BM83 -> Nightwave:Microchip_BM83_GroundLands; symbol RF_Bluetooth:Microchip_BM83 -> Nightwave:U12
Connections:
- net +3V6_BT: now also U12.23 (BAT_IN), C36.1 (+3V6_BT), C37.1 (+3V6_BT)
- net BT_LED: now also U12.32 (LED1); no longer U12.7 (AOHPM), U12.8 (AOHPL)
- net BT_MCLK_OPTION: now also U12.5 (MCLK1); no longer U12.37 (DP)
- net BT_MFB: now also U12.26 (PWR(MFB)); no longer U12.1 (DR1), U12.2 (RFS1)
- net BT_RST_N: now also U12.43 (~{RST}); no longer U12.28 (SK2_KEY_AD)
- net BT_SERVICE_P34: now also U12.31 (P3_4/UART_RTS); no longer U12.45 (P0_7)
- net BT_UART_RX: now also U12.30 (P8_5/UART_TXD); no longer U12.40 (P0_5)
- net BT_UART_TX: now also U12.29 (P8_6/UART_RXD); no longer U12.38 (P0_3)
- net BT_WAKE: now also U12.49 (P0_0/UART_TX_IND); no longer U12.32 (LED1)
- net GND: now also U12.16 (GND), U12.50 (GND), U12.56 (GND), U12.57 (GND), C36.2 (GND), C37.2 (GND)
- net I2S_BCLK: now also R13.1 (I2S_BCLK); no longer R13.2
- net I2S_BCLK_BT: now also R13.2 (I2S_BCLK_BT), U12.3 (SCLK1); no longer R13.1, R14.1, R15.1, U12.26 (PWR(MFB)), U12.27 (SK1_AMB_DET)
- net I2S_DOUT: now also R15.1 (I2S_DOUT); no longer R15.2
- net I2S_LRCLK: now also R14.1 (I2S_LRCLK); no longer R14.2
- net BT_STATE: now reaches U12.34 (LED2)
- net I2C_SCL: no longer names the net of U12.20 (P3_2)
- net I2C_SDA: no longer names the net of U12.39 (P2_7)
- new net I2S_DOUT_BT: R15.2 (I2S_DOUT_BT), U12.1 (DR1)
- new net I2S_LRCLK_BT: R14.2 (I2S_LRCLK_BT), U12.2 (RFS1)
- no-connect marks 31 -> 35
